Commit message: Weld the Franka meshes into GLB to reduce the urdf layer size
Co-Authored-By: Claude Fable 5 <noreply@anthropic.com>

File: examples/libero/urdf/fer/fer.urdf (robot description, URDF)
Before this commit: robot fer, 14 links, 13 joints
Links:
- link fer_hand: geometry visual mesh filename=meshes/robot_ee/franka_hand_white/visual/hand.glb
- link fer_leftfinger: geometry visual mesh filename=meshes/robot_ee/franka_hand_white/visual/finger.glb
- link fer_link0: geometry visual mesh filename=meshes/robots/fer/visual/link0.glb
- link fer_link1: geometry visual mesh filename=meshes/robots/fer/visual/link1.glb
- link fer_link2: geometry visual mesh filename=meshes/robots/fer/visual/link2.glb
- link fer_link3: geometry visual mesh filename=meshes/robots/fer/visual/link3.glb
- link fer_link4: geometry visual mesh filename=meshes/robots/fer/visual/link4.glb
- link fer_link5: geometry visual mesh filename=meshes/robots/fer/visual/link5.glb
- link fer_link6: geometry visual mesh filename=meshes/robots/fer/visual/link6.glb
- link fer_link7: geometry visual mesh filename=meshes/robots/fer/visual/link7.glb
- link fer_rightfinger: geometry visual mesh filename=meshes/robot_ee/franka_hand_white/visual/finger.glb
